Commit message: B

File: model/robot.xacro (robot description, xacro)
@@ -1,174 +1,116 @@
-<robot name="ddmr" xmlns:xacro="http://www.ros.org/wiki/xacro">
-<!-- start of properties definition-->
-  <xacro:property name="PI" value="3.14159"/>
-  <xacro:property name="DIV_CM" value="0.01"/>
-  <!--body-->
-  <xacro:property name="body_length" value="${16 * DIV_CM}"/>  <!-- a -->
-  <xacro:property name="body_height" value="${6 * DIV_CM}"/>  <!-- b -->
-  <xacro:property name="body_width" value="${14 * DIV_CM}"/>  <!-- c -->
-  <!--wheel & caster-->
-  <xacro:property name="r" value="${5 * DIV_CM}"/> <!-- radius -->
-  <xacro:property name="d" value="${1 * DIV_CM}"/> <!-- wheel thickness, not caster -->
-  <xacro:property name="ori_to_ground" value="${body_height / 2 + r}"/>  <!-- s1 -->
-  <xacro:property name="ori_to_wheels" value="${2 * r}"/>  <!-- s2 -->
-  <xacro:property name="ori_to_caster" value="${2 * r}"/>  <!-- s3 -->
-  <xacro:property name="mid_to_wheels" value="${body_width / 2 + d/2}"/>  <!-- s4 -->
-  <!--
-    BODY (cuboid)
-  Volume = body_width * body_length * body_height
-  mass = density * volume
-  moment of inertia (Ix) = mass * (body_height^2 + body_width^2) / 12
-  moment of inertia (Iy) = mass * (body_length^2 + body_height^2) / 12
-  moment of inertia (Iz) = mass * (body_length^2 + body_width^2) / 12
-    WHEEL (Cylinder)
-  volume = PI * r^2 * d
-  mass = density * volume
-  moment of inertia (Ix) = (1/12) * mass * (3 * r^2 + d^2)
-  moment of inertia (Iy) = (1/12) * mass * (3 * r^2 + d^2)
-  moment of inertia (Iz) = (1/2) * mass * (r^2 + d^2)
-    CASTER (Ball)
-  volume = (4/3) * PI * (r/2)^3
-  mass = density * volume
-  moment of inertia (Ix) = (2/5) * mass * (r/2)^2
-  moment of inertia (Iy) = (2/5) * mass * (r/2)^2
-  moment of inertia (Iz) = (2/5) * mass * (r/2)^2
-  -->
-  <!-- Densities (kg/m^3) -->
-  <xacro:property name="body_density" value="2710"/>
-  <xacro:property name="wheels_density" value="2710"/>
-  <xacro:property name="caster_density" value="2710"/>
-  <!-- Masses -->
-  <xacro:property name="body_mass" value="${body_density * body_length * body_height * body_width}"/>
-  <xacro:property name="wheel_mass" value="${wheels_density * PI * r**2 * d}"/>
-  <xacro:property name="caster_mass"  value="${caster_density * (4.0/3.0) * PI * (r/2)**3}"/>
-  <!-- Moments of inertia -->
-  <xacro:property name="body_ix" value="${body_mass * (body_height**2 + body_width**2) / 12}"/>
-  <xacro:property name="body_iy" value="${body_mass * (body_length**2 + body_height**2) / 12}"/>
-  <xacro:property name="body_iz" value="${body_mass * (body_length**2 + body_width**2) / 12}"/>
-  <xacro:property name="wheel_ixy" value="${(1.0/12.0) * wheel_mass * (3 * r**2 + d**2)}"/>
-  <xacro:property name="wheel_iz" value="${(1.0/2.0) * wheel_mass * (r**2)}"/>
-  <xacro:property name="caster_ixyz" value="${caster_mass * (2.0/5.0) * (r/2)**2}"/>
-<!-- end of properties definition-->
-<!-- CoM C2 (body) CoM C1 (projection from C2 to ground) -->
-<!-- -->
+<?xml version="1.0"?>
+<robot name="differential_drive_robot" xmlns:xacro="http://www.ros.org/wiki/xacro">
+  <xacro:property name="pi_const" value="3.14159265"/>
+  <xacro:property name="a" value="1" />
+  <xacro:property name="b" value="0.3" />
+  <xacro:property name="c" value="0.6"/>
+  <xacro:property name="r" value="0.15"/>
+  <xacro:property name="d" value="0.1"/>
+  <xacro:property name="s1" value="${b/2+r}"/>
+  <xacro:property name="s2" value="${2*r}"/>
+  <xacro:property name="s3" value="${2*r}"/>
+  <xacro:property name="s4" value="${c/2+d/2}"/>
+  <xacro:property name="d1" value="2710.0"/>
+  <xacro:property name="d2" value="2710.0"/>
+  <xacro:property name="d3" value="2710.0"/>
+  <xacro:property name="m1" value="${d1*a*b*c}"/>
+  <xacro:property name="m2" value="${d2*pi_const*r*r*d}"/>
+  <xacro:property name="m3" value="${d3*(4.0/3.0)*pi_const*r*r*r}"/>
+  <!-- Moments of inertia of the robot body -->
+  <xacro:property name="Ix_body" value="${(1/12)*m1*(b*b+c*c)}"/>
+  <xacro:property name="Iy_body" value="${(1/12)*m1*(a*a+b*b)}"/>
+  <xacro:property name="Iz_body" value="${(1/12)*m1*(a*a+c*c)}"/>
+  <!-- Moments of inertia of the wheels -->
+  <xacro:property name="Iz_wheel" value="${0.5*m2*r*r}"/>
+  <xacro:property name="I_wheel" value="${(1.0/12.0)*m2*(3.0*r*r+d*d)}"/>
+  <!-- Moments of inertia of the caster sphere -->
+  <xacro:property name="I_caster" value="${(2.0/5.0)*m3*r*r}"/>
 <xacro:macro name="inertia_body">
-    <inertial>
-        <origin rpy="0 0 0" xyz="0 0 ${ori_to_ground}"/> <!-- rpy (roll, pitch, yaw) -->
-        <mass value="${body_mass}"/>
-        <inertia ixx="${body_ix}" ixy="0.0" ixz="0.0" iyy="${body_iy}" iyz="0.0" izz="${body_iz}"/>
-    </inertial>
+  <inertial>
+    <origin rpy="0 0 0" xyz="0 0 ${s1}"/>
+    <mass value="${m1}"/>
+    <inertia ixx="${Ix_body}" ixy="0.0" ixz="0.0" iyy="${Iy_body}" iyz="0" izz="${Iz_body}" />
+  </inertial>
 </xacro:macro>
-<!-- CoM C5(wheel1) C4(wheel2) -->
-<xacro:macro name="inertia_wheel">
-    <inertial>
+  <xacro:macro name="inertia_wheel">
+  <inertial>
+    <origin rpy="1.570795 0 0" xyz="0 0 0"/>
+    <mass value="${m2}"/>
+    <inertia ixx="${I_wheel}" ixy="0.0" ixz="0.0" iyy="${I_wheel}" iyz="0" izz="${Iz_wheel}" />
+  </inertial>
+</xacro:macro>
+  <xacro:macro name="inertia_caster">
+  <inertial>
     <origin rpy="0 0 0" xyz="0 0 0"/>
-        <mass value="${wheel_mass}"/>
-    <inertia ixx="${wheel_ixy}" ixy="0.0" ixz="0.0" iyy="${wheel_iz}" iyz="0.0" izz="${wheel_ixy}"/>
-    </inertial>
-</xacro:macro>
-<!-- CoM C3 (caster) -->
-<xacro:macro name="inertia_caster">
-    <inertial>
-    <origin rpy="0 0 0" xyz="0 0 0"/>
-        <mass value="${caster_mass}"/>
-        <inertia ixx="${caster_ixyz}" ixy="0.0" ixz="0.0" iyy="${caster_ixyz}" iyz="0.0" izz="${caster_ixyz}"/>
-    </inertial>
-</xacro:macro>
-<!-- Files Includes-->
-<xacro:include filename="$(find mobile_robot)/model/robot.gazebo"/>
-<!--START Links andd joints body-->
-    <link name="base_footprint"> </link>
-    <joint name="body_link_joint" type="fixed">
-        <parent link="base_footprint"/>
-        <child link="body_link"/>
-    </joint>
-    <link name="body_link">
-        <visual>
-            <geometry>
-                <box size="${body_length} ${body_width} ${body_height}"/>
-            </geometry>
-            <origin rpy="0 0 0" xyz="0 0 ${ori_to_ground}"/>
-    <!--        <material name="blue">
-                <color rgba="0 0 1 1"/>
-            </material> //forlater    -->
-        </visual>
-        <collision>
-            <geometry>
-                <box size="${body_length} ${body_width} ${body_height}"/>
-            </geometry>
-            <origin rpy="0 0 0" xyz="0 0 ${ori_to_ground}"/>
-        </collision>
-        <xacro:inertia_body/>
-    </link>
-<!--END Links andd joints body-->
-<!-- START -->
-<joint name="wheel_joint" type="continuous">
-  <parent link="body_link"/>
-  <child link="wheel_link"/>
-  <origin xyz="${-ori_to_wheels} ${-mid_to_wheels} ${r}" rpy="0 0 0"/> <!-- s2 s4 -->
-  <axis xyz="0 1 0"/>
-  <limit effort="50000" velocity="10"/>
-  <dynamics damping="1.0" friction="1.0"/>
-</joint>
-<link name="wheel_link">
-  <visual>
-    <origin xyz="0 0 0" rpy="1.570795 0 0"/>
-    <geometry>
-      <cylinder length="${d}" radius="${r}"/>
-    </geometry>
-  </visual>
-  <collision>
-    <origin xyz="0 0 0" rpy="1.570795 0 0"/>
-    <geometry>
-      <cylinder length="${d}" radius="${r}"/>
-    </geometry>
-  </collision>
-  <xacro:inertia_wheel/>
-</link>
-<!-- END -->
-<!-- START -->
-<joint name="wheel2_joint" type="continuous">
-  <parent link="body_link"/>
-  <child link="wheel2_link"/>
-  <origin xyz="${-ori_to_wheels} ${mid_to_wheels} ${r}" rpy="0 0 0"/>
-  <axis xyz="0 1 0"/>
-  <limit effort="50000" velocity="10"/>
-  <dynamics damping="1.0" friction="1.0"/>
-</joint>
-<link name="wheel2_link">
-  <visual>
-    <origin xyz="0 0 0" rpy="1.570795 0 0"/>
-    <geometry>
-      <cylinder length="${d}" radius="${r}"/>
-    </geometry>
-  </visual>
-  <collision>
-    <origin xyz="0 0 0" rpy="1.570795 0 0"/>
-    <geometry>
-      <cylinder length="${d}" radius="${r}"/>
-    </geometry>
-  </collision>
-  <xacro:inertia_wheel/>
-</link>
-<!-- END -->
-<!-- START caster -->
-<joint name="caster_joint" type="fixed">
-  <parent link="body_link"/>
-  <child link="caster_link"/>
-  <origin xyz="${ori_to_wheels} 0 ${r / 2}" rpy="0 0 0"/>
-</joint>
-<link name="caster_link">
-  <visual>
-    <geometry>
-      <sphere radius="${r / 2}"/>
-    </geometry>
-  </visual>
-  <collision>
-    <geometry>
-      <sphere radius="${r / 2}"/>
-    </geometry>
-  </collision>
-  <xacro:inertia_caster/>
-</link>
-<!-- END caster -->
+    <mass value="${m3}"/>
+    <inertia ixx="${I_caster}" ixy="0.0" ixz="0.0" iyy="${I_caster}" iyz="0" izz="${I_caster}" />
+  </inertial>
+  </xacro:macro>
+  <xacro:include filename="$(find mobile_robot)/model/robot.gazebo"/>
+  <link name="base_footprint"/>
+  <joint name="body_link_joint" type="fixed">
+    <parent link="base_footprint"/>
+    <child link="body_link"/>
+  </joint>
+  <link name="body_link">
+    <visual>
+      <geometry>
+        <box size="${a} ${c} ${b}"/>
+      </geometry>
+      <origin rpy="0 0 0" xyz="0 0 ${s1}"/>
+    </visual>
+    <collision>
+      <geometry>
+        <box size="${a} ${c} ${b}"/>
+      </geometry>
+      <origin rpy="0 0 0" xyz="0 0 ${s1}"/>
+    </collision>
+    <xacro:inertia_body/>
+  </link>
+  <joint name="wheel1_joint" type="continuous">
+    <parent link="body_link"/>
+    <child link="wheel1_link"/>
+    <origin xyz="${-s2} ${-s4} ${r}" rpy="0 0 0"/>
+    <axis xyz="0 1 0"/>
+    <limit effort="50000" velocity="10"/>
+    <dynamics damping="1.0" friction="1.0"/>
+  </joint>
+  <link name="wheel1_link">
+    <visual>
+      <origin rpy="1.570795 0 0" xyz="0 0 0"/>
+      <geometry>
+        <cylinder length="${d}" radius="${r}"/>
+      </geometry>
+    </visual>
+    <collision>
+      <origin rpy="1.570795 0 0" xyz="0 0 0"/>
+      <geometry>
+        <cylinder length="${d}" radius="${r}"/>
+      </geometry>
+    </collision>
+    <xacro:inertia_wheel/>
+  </link>
+  <joint name="wheel2_joint" type="continuous">
+    <parent link="body_link"/>
+    <child link="wheel2_link"/>
+    <origin xyz="${-s2} ${s4} ${r}" rpy="0 0 0"/>
+    <axis xyz="0 1 0"/>
+    <limit effort="50000" velocity="10"/>
+    <dynamics damping="1.0" friction="1.0"/>
+  </joint>
+  <link name="wheel2_link">
+    <visual>
+      <origin rpy="1.570795 0 0" xyz="0 0 0"/>
+      <geometry>
+        <cylinder length="${d}" radius="${r}"/>
+      </geometry>
+    </visual>
+    <collision>
+      <origin rpy="1.570795 0 0" xyz="0 0 0"/>
+      <geometry>
+        <cylinder length="${d}" radius="${r}"/>
+      </geometry>
+    </collision>
+    <xacro:inertia_wheel/>
+  </link>
 </robot>
